Commit message: Update model.urdf

File: model.urdf (robot description, URDF)
Before this commit: robot converted_robot, 8 links, 0 joints
Links:
- removed link legs
- removed link raspi_btm
- removed link raspi_top
- removed link rotor_0
- removed link rotor_1
- removed link rotor_2
- removed link rotor_3
- link base_link: geometry visual mesh filename=model://base_link.stl scale=0.001 0.001 0.001

Commit message: Update model.urdf

File: model.urdf (robot description, URDF)
Before this commit: robot acds_quad_base, 1 links, 0 joints
Links:
- link base_link: mass None -> 0.6477; geometry collision mesh filename=base_link.stl scale=0.001 0.001 0.001; visual mesh filename=base_link.stl scale=0.001 0.001 0.001

Commit message: Update model.urdf

File: model.urdf (robot description, URDF)
Before this commit: robot acds_quad_base, 1 links, 0 joints
Links:
- link base_link: mass 0.6477 -> None

Commit message: Update model.urdf

File: model.urdf (robot description, URDF)
Before this commit: robot acds_quad_base, 1 links, 0 joints
Links:
- added link legs; collision mesh filename=legs.stl scale=0.001 0.001 0.001; visual mesh filename=legs.stl scale=0.001 0.001 0.001
Joints:
- added joint joint_legs: type fixed, parent , child , origin xyz=0.07111352813714546 0.10450989979429313 0.016522611625440435 rpy=0 0.2618 -1.5707963267948966

Commit message: Update model.urdf

File: model.urdf (robot description, URDF)
Before this commit: robot acds_quad_base, 2 links, 1 joints
Links:
- removed link legs
Joints:
- removed joint joint_legs
